File: custom-pcb.kicad_sch (KiCad schematic)
At the start: 161 parts, among them J1 USB_C_Receptacle, SW1 SW_SPDT, U1 AMS1117-3.3, U2 STM32F072CBT6, Y1 16MHz (10p)

Commit message: Cleanup
Changed lines of the file:
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@@
   (junction (at 185.42 55.88) (diameter 0) (color 0 0 0 0)
   )
+  (junction (at 203.2 49.53) (diameter 0) (color 0 0 0 0)
+  )
   (junction (at 248.92 209.55) (diameter 0) (color 0 0 0 0)
   )
@@
   (junction (at 53.34 193.04) (diameter 0) (color 0 0 0 0)
   )
+  (junction (at 41.91 46.99) (diameter 0) (color 0 0 0 0)
+  )
   (junction (at 248.92 242.57) (diameter 0) (color 0 0 0 0)
   )
@@
   (no_connect (at 203.2 105.41))
   (no_connect (at 203.2 107.95))
-  (no_connect (at 203.2 111.76))
+  (no_connect (at 203.2 110.49))
   (no_connect (at 203.2 113.03))
   (no_connect (at 203.2 115.57))
@@
     (stroke (width 0) (type default) (color 0 0 0 0))
   )
+  (wire (pts (xy 41.91 46.99) (xy 43.18 46.99))
+    (stroke (width 0) (type default) (color 0 0 0 0))
+  )
   (wire (pts (xy 95.25 193.04) (xy 109.22 193.04))
     (stroke (width 0) (type default) (color 0 0 0 0))
@@
     (stroke (width 0) (type default) (color 0 0 0 0))
   )
-  (wire (pts (xy 195.58 49.53) (xy 207.01 49.53))
+  (wire (pts (xy 195.58 49.53) (xy 203.2 49.53))
     (stroke (width 0) (type default) (color 0 0 0 0))
   )
@@
     (stroke (width 0) (type default) (color 0 0 0 0))
   )
+  (wire (pts (xy 203.2 49.53) (xy 207.01 49.53))
+    (stroke (width 0) (type default) (color 0 0 0 0))
+  )
   (wire (pts (xy 151.13 187.96) (xy 153.67 187.96))
     (stroke (width 0) (type default) (color 0 0 0 0))
@@
     (stroke (width 0) (type default) (color 0 0 0 0))
   )
-  (wire (pts (xy 36.83 46.99) (xy 43.18 46.99))
+  (wire (pts (xy 36.83 46.99) (xy 41.91 46.99))
     (stroke (width 0) (type default) (color 0 0 0 0))
   )
@@
     (pin "2")
   )
+  (symbol (lib_id "power:PWR_FLAG") (at 203.2 49.53 0) (unit 1)
+    (in_bom yes) (on_board yes)
+    (property "Reference" "#FLG0101" (id 0) (at 203.2 47.625 0)
+      (effects (font (size 1.27 1.27)) hide)
+    )
+    (property "Value" "PWR_FLAG" (id 1) (at 203.2 45.72 0))
+    (property "Footprint" "" (id 2) (at 203.2 49.53 0)
+      (effects (font (size 1.27 1.27)) hide)
+    )
+    (property "Datasheet" "~" (id 3) (at 203.2 49.53 0)
+      (effects (font (size 1.27 1.27)) hide)
+    )
+    (pin "1")
+  )
   (symbol (lib_id "MX_Alps_Hybrid:MX-NoLED") (at 127 217.17 0) (unit 1)
     (in_bom yes) (on_board yes)
@@
     (pin "1")
   )
+  (symbol (lib_id "power:PWR_FLAG") (at 50.8 57.15 180) (unit 1)
+    (in_bom yes) (on_board yes)
+    (property "Reference" "#FLG0103" (id 0) (at 50.8 59.055 0)
+      (effects (font (size 1.27 1.27)) hide)
+    )
+    (property "Value" "PWR_FLAG" (id 1) (at 50.8911 60.5068 0)
+      (effects (font (size 1 1)))
+    )
+    (property "Footprint" "" (id 2) (at 50.8 57.15 0)
+      (effects (font (size 1.27 1.27)) hide)
+    )
+    (property "Datasheet" "~" (id 3) (at 50.8 57.15 0)
+      (effects (font (size 1.27 1.27)) hide)
+    )
+    (pin "1")
+  )
   (symbol (lib_id "Device:D_Small") (at 53.34 190.5 90) (unit 1)
     (in_bom yes) (on_board yes)
@@
     (pin "2")
   )
+  (symbol (lib_id "power:PWR_FLAG") (at 41.91 46.99 0) (unit 1)
+    (in_bom yes) (on_board yes)
+    (property "Reference" "#FLG0102" (id 0) (at 41.91 45.085 0)
+      (effects (font (size 1.27 1.27)) hide)
+    )
+    (property "Value" "PWR_FLAG" (id 1) (at 41.8189 43.6332 0)
+      (effects (font (size 1 1)))
+    )
+    (property "Footprint" "" (id 2) (at 41.91 46.99 0)
+      (effects (font (size 1.27 1.27)) hide)
+    )
+    (property "Datasheet" "~" (id 3) (at 41.91 46.99 0)
+      (effects (font (size 1.27 1.27)) hide)
+    )
+    (pin "1")
+  )
   (symbol (lib_id "Device:C_Small") (at 119.38 111.76 0) (unit 1)
     (in_bom yes) (on_board yes) (fields_autoplaced)
@@
   )
   (symbol_instances
+    (path "/2d7bbcf3-87ca-44cf-a5d0-4beb50d51251"
+      (reference "#FLG0101") (unit 1) (value "PWR_FLAG") (footprint "")
+    )
+    (path "/79433de7-1e65-4dbd-97fc-4c7030c08088"
+      (reference "#FLG0102") (unit 1) (value "PWR_FLAG") (footprint "")
+    )
+    (path "/6a03a94d-bb8c-41ef-816d-79304f6fb241"
+      (reference "#FLG0103") (unit 1) (value "PWR_FLAG") (footprint "")
+    )
     (path "/d32eea30-5e68-4ff3-b5cb-57f4fc80e4d1"
       (reference "#PWR0101") (unit 1) (value "GND") (footprint "")
